Commit message: rdy 4 submission

File: catkin_ws/src/my_robot/urdf/my_robot.xacro (robot description, xacro)
@@ -9,5 +9,4 @@
     </joint>
     <link name='chassis'>
-    <pose>0 0 0.1 0 0 0</pose>
     <inertial>
         <mass value="15.0"/>
@@ -22,5 +21,5 @@
         <origin xyz="0 0 0" rpy=" 0 0 0"/>
         <geometry>
-        <box size=".39 .25 .12"/>
+        <cylinder length="0.10" radius="0.20"/>
         </geometry>
     </collision>
@@ -28,9 +27,9 @@
         <origin xyz="0 0 0" rpy=" 0 0 0"/>
         <geometry>
-        <box size=".39 .25 .12"/>
+        <cylinder length="0.10" radius="0.20"/>
         </geometry>
     </visual>
     <collision name='back_caster_collision'>
-        <origin xyz="-0.14 0 -0.06" rpy=" 0 0 0"/>
+        <origin xyz="-0.1 0 -0.06" rpy=" 0 0 0"/>
         <geometry>
         <sphere radius="0.0499"/>
@@ -38,5 +37,5 @@
     </collision>
     <visual name='back_caster_visual'>
-        <origin xyz="-0.14 0 -0.06" rpy=" 0 0 0"/>
+        <origin xyz="-0.1 0 -0.06" rpy=" 0 0 0"/>
         <geometry>
         <sphere radius="0.05"/>
@@ -44,5 +43,5 @@
     </visual>
     <collision name='front_caster_collision'>
-        <origin xyz="0.14 0 -0.06" rpy=" 0 0 0"/>
+        <origin xyz="0.1 0 -0.06" rpy=" 0 0 0"/>
         <geometry>
         <sphere radius="0.0499"/>
@@ -50,5 +49,5 @@
     </collision>
     <visual name='front_caster_visual'>
-        <origin xyz="0.14 0 -0.06" rpy=" 0 0 0"/>
+        <origin xyz="0.1 0 -0.06" rpy=" 0 0 0"/>
         <geometry>
         <sphere radius="0.05"/>
@@ -57,62 +56,62 @@
     </link>
     <link name='left_wheel'>
-    <inertial>
-        <mass value="5.0"/>
-        <origin xyz="0.0 0 0" rpy=" 0 1.5707 1.5707"/>
-        <inertia
-            ixx="0.1" ixy="0" ixz="0"
-            iyy="0.1" iyz="0"
-            izz="0.1"
-        />
-    </inertial>
-    <collision name='left_wheel_collision'>
-        <origin xyz="0 0 0" rpy=" 0 1.5707 1.5707"/>
-        <geometry>
-        <cylinder radius="0.12" length="0.05"/>
-        </geometry>
-    </collision>
-    <visual name='left_wheel_visual'>
-        <origin xyz="0 0 0" rpy=" 0 1.5707 1.5707"/>
-        <geometry>
-        <cylinder radius="0.12" length="0.05"/>
-        </geometry>
-    </visual>
+        <inertial>
+            <mass value="5.0"/>
+            <origin xyz="0 0 0" rpy=" 0 0 0"/>
+            <inertia
+                ixx="0.01" ixy="0" ixz="0"
+                iyy="0.01" iyz="0"
+                izz="0.01"
+            />
+        </inertial>
+        <collision name='left_wheel_collision'>
+            <origin xyz="0 0 0" rpy=" 0 1.5707 1.5707"/>
+            <geometry>
+            <cylinder radius="0.12" length="0.05"/>
+            </geometry>
+        </collision>
+        <visual name='left_wheel_visual'>
+            <origin xyz="0 0 0" rpy=" 0 1.5707 1.5707"/>
+            <geometry>
+            <cylinder radius="0.12" length="0.05"/>
+            </geometry>
+        </visual>
     </link>
     <link name='right_wheel'>
-    <inertial>
-        <mass value="5.0"/>
-        <origin xyz="0.0 0 0" rpy=" 0 1.5707 1.5707"/>
-        <inertia
-            ixx="0.1" ixy="0" ixz="0"
-            iyy="0.1" iyz="0"
-            izz="0.1"
-        />
-    </inertial>
-    <collision name='right_wheel_collision'>
-        <origin xyz="0 0 0" rpy=" 0 1.5707 1.5707"/>
-        <geometry>
-        <cylinder radius="0.12" length="0.05"/>
-        </geometry>
-    </collision>
-    <visual name='right_wheel_visual'>
-        <origin xyz="0 0 0" rpy=" 0 1.5707 1.5707"/>
-        <geometry>
-        <cylinder radius="0.12" length="0.05"/>
-        </geometry>
-    </visual>
+        <inertial>
+            <mass value="5.0"/>
+            <origin xyz="0 0 0" rpy=" 0 0 0"/>
+            <inertia
+                ixx="0.01" ixy="0" ixz="0"
+                iyy="0.01" iyz="0"
+                izz="0.01"
+            />
+        </inertial>
+        <collision name='right_wheel_collision'>
+            <origin xyz="0 0 0" rpy=" 0 1.5707 1.5707"/>
+            <geometry>
+            <cylinder radius="0.12" length="0.05"/>
+            </geometry>
+        </collision>
+        <visual name='right_wheel_visual'>
+            <origin xyz="0 0 0" rpy=" 0 1.5707 1.5707"/>
+            <geometry>
+            <cylinder radius="0.12" length="0.05"/>
+            </geometry>
+        </visual>
     </link>
     <joint type="continuous" name="left_wheel_hinge">
-        <origin xyz="0 0.175 0" rpy="0 0 0"/>
+        <origin xyz="0 0.225 0" rpy="0 0 0"/>
         <child link="left_wheel"/>
         <parent link="chassis"/>
-        <axis xyz="0 1 0" rpy="0 0 0"/>
+        <axis xyz="0 1 0"/>
         <limit effort="10000" velocity="1000"/>
         <dynamics damping="1.0" friction="1.0"/>
     </joint>
     <joint type="continuous" name="right_wheel_hinge">
-        <origin xyz="0 -0.175 0" rpy="0 0 0"/>
+        <origin xyz="0 -0.225 0" rpy="0 0 0"/>
         <child link="right_wheel"/>
         <parent link="chassis"/>
-        <axis xyz="0 1 0" rpy="0 0 0"/>
+        <axis xyz="0 1 0"/>
         <limit effort="10000" velocity="1000"/>
         <dynamics damping="1.0" friction="1.0"/>
@@ -128,4 +127,10 @@
             />
         </inertial>
+        <collision name="camera_collision">
+            <origin xyz="0 0 0" rpy="0 0 0"/>
+            <geometry>
+                <box size="0.05 0.05 0.05"/>
+            </geometry>
+        </collision>
         <visual name="camera_visual">
             <origin xyz="0 0 0" rpy="0 0 0"/>
@@ -134,16 +139,9 @@
             </geometry>
         </visual>
-        <collision name="camera_collision">
-            <origin xyz="0 0 0" rpy="0 0 0"/>
-            <geometry>
-                <box size="0.05 0.05 0.05"/>
-            </geometry>
-        </collision>
     </link>
-    <joint name="camera_joint" type="fixed">
-        <origin xyz="0.195 0 0.0" rpy="0 0 0"/>
-        <axis xyz="0 1 0"/>
+    <joint type="fixed" name="camera_joint">
+        <origin xyz="0.20 0 0.0" rpy="0 0 0"/>
+        <child link="camera"/>
         <parent link="chassis"/>
-        <child link="camera"/>
     </joint>
     <joint name="camera_optical_joint" type="fixed">
@@ -152,6 +150,6 @@
         <child link="camera_link_optical"/>
     </joint>
-  <link name="camera_link_optical">
-  </link>
+    <link name="camera_link_optical">
+    </link>
     <link name="hokuyo">
         <inertial>
@@ -178,6 +176,5 @@
     </link>
     <joint name="hokuyo_joint" type="fixed">
-        <origin xyz="0.145 0 0.12" rpy="0 0 0"/>
-        <axis xyz="0 1 0"/>
+        <origin xyz="0.15 0 0.10" rpy="0 0 0"/>
         <parent link="chassis"/>
         <child link="hokuyo"/>
@@ -195,3 +192,6 @@
         <material>Gazebo/Green</material>
     </gazebo>
+    <gazebo reference="hokuyo">
+        <material>Gazebo/Green</material>
+    </gazebo>
 </robot>
